File: project/ECAD/emilien version 25 03 2026.kicad_pcb (KiCad board)
At the start: 2 copper layers, 81.5 x 57.8 mm, 20 parts, among them J1 Barrel_Jack_Switch, J2 Moteur 1, J3 Moteur 2, J4 limit switch x, J5 limit switch y, J6 SD_Card_Device, J7 Ecran, U1 ESP32-S3-UNO, U2 R-78E5.0-1.0

Commit message: fix some wiring problems
Connections:
- C6 pad 1: +5V -> +12V
- U1 pad 8: +5V -> +12V
Routing:
- net +5V: track 111.9 -> 3.58 mm
- net +12V: track 92.7 -> 145.2 mm
Changed lines of the file:
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@@
 			(unit
 				(name "A")
-				(pins "20" "19" "1" "3" "9" "10" "11" "12" "13" "14" "8" "2" "7" "6"
-					"29" "4" "16" "15" "30" "32" "31" "28" "27" "26" "25" "24" "23" "22"
+				(pins "20" "19" "1" "3" "9" "10" "11" "12" "13" "14" "8" "2" "6" "29"
+					"7" "4" "16" "15" "30" "32" "31" "28" "27" "26" "25" "24" "23" "22"
 					"21" "18" "17"
 				)
@@
 			(layers "*.Cu" "*.Mask")
 			(remove_unused_layers no)
-			(net "+5V")
+			(net "+12V")
 			(pinfunction "VIN_8")
 			(pintype "power_in")
@@
 			(layers "F.Cu" "F.Mask" "F.Paste")
 			(roundrect_rratio 0.217391)
-			(net "+5V")
+			(net "+12V")
 			(pintype "passive")
 		)
@@
 			(keep_text_aligned yes)
 		)
-		(gr_text "57,0542"
+		(gr_text "57.0542"
 			(at 214.299959 97.527104 90)
 			(layer "User.1")
@@
 			(keep_text_aligned yes)
 		)
-		(gr_text "81,4811"
+		(gr_text "81.4811"
 			(at 154.780532 59.85 0)
 			(layer "User.1")
@@
 	)
 	(segment
-		(start 137.125 77.7)
-		(end 137.125 78)
-		(width 1)
-		(layer "F.Cu")
-		(net "+5V")
-	)
-	(segment
-		(start 118 109.6)
-		(end 166.97 109.6)
-		(width 1)
-		(layer "F.Cu")
-		(net "+5V")
-	)
-	(segment
-		(start 116.8 92.8)
-		(end 116.8 108.4)
-		(width 1)
-		(layer "F.Cu")
-		(net "+5V")
-	)
-	(segment
-		(start 172.985 115.225)
-		(end 176.29 115.225)
-		(width 1)
-		(layer "F.Cu")
-		(net "+5V")
-	)
-	(segment
-		(start 138.45 82.171321)
-		(end 137.421321 83.2)
-		(width 1)
-		(layer "F.Cu")
-		(net "+5V")
-	)
-	(segment
-		(start 137.125 78)
-		(end 137.125 79.125)
-		(width 1)
-		(layer "F.Cu")
-		(net "+5V")
-	)
-	(segment
-		(start 166.97 109.6)
-		(end 172.79 115.42)
-		(width 1)
-		(layer "F.Cu")
-		(net "+5V")
-	)
-	(segment
-		(start 137.12 77.695)
-		(end 137.125 77.7)
-		(width 1)
-		(layer "F.Cu")
-		(net "+5V")
-	)
-	(segment
-		(start 126.4 83.2)
-		(end 116.8 92.8)
-		(width 1)
-		(layer "F.Cu")
-		(net "+5V")
-	)
-	(segment
-		(start 137.125 79.125)
-		(end 138.45 80.45)
-		(width 1)
-		(layer "F.Cu")
-		(net "+5V")
-	)
-	(segment
-		(start 172.79 115.42)
-		(end 172.985 115.225)
-		(width 1)
-		(layer "F.Cu")
-		(net "+5V")
-	)
-	(segment
-		(start 116.8 108.4)
-		(end 118 109.6)
-		(width 1)
-		(layer "F.Cu")
-		(net "+5V")
-	)
-	(segment
-		(start 138.45 80.45)
-		(end 138.45 82.171321)
-		(width 1)
-		(layer "F.Cu")
-		(net "+5V")
-	)
-	(segment
-		(start 137.421321 83.2)
-		(end 126.4 83.2)
-		(width 1)
-		(layer "F.Cu")
-		(net "+5V")
-	)
-	(segment
-		(start 137.12 74.99)
-		(end 137.12 77.695)
-		(width 1)
-		(layer "F.Cu")
-		(net "+5V")
-	)
-	(segment
 		(start 124.25 97.51)
 		(end 124.29 97.55)
@@
 	)
 	(segment
+		(start 117.5 96)
+		(end 117.5 100.55)
+		(width 1.5)
+		(layer "F.Cu")
+		(net "+12V")
+	)
+	(segment
 		(start 172.79 120.5)
 		(end 172.29 120.5)
@@
 	)
 	(segment
+		(start 139 79.875)
+		(end 139 84)
+		(width 1.5)
+		(layer "F.Cu")
+		(net "+12V")
+	)
+	(segment
+		(start 137.125 78)
+		(end 139 79.875)
+		(width 1.5)
+		(layer "F.Cu")
+		(net "+12V")
+	)
+	(segment
+		(start 117.42 90.08)
+		(end 117.42 95.92)
+		(width 1.5)
+		(layer "F.Cu")
+		(net "+12V")
+	)
+	(segment
+		(start 117.42 95.92)
+		(end 117.5 96)
+		(width 1.5)
+		(layer "F.Cu")
+		(net "+12V")
+	)
+	(segment
+		(start 136.5 86.5)
+		(end 121 86.5)
+		(width 1.5)
+		(layer "F.Cu")
+		(net "+12V")
+	)
+	(segment
 		(start 136.95 94.25)
 		(end 136.95 96.65)
@@
 	)
 	(segment
+		(start 139 84)
+		(end 136.5 86.5)
+		(width 1.5)
+		(layer "F.Cu")
+		(net "+12V")
+	)
+	(segment
 		(start 152.04 107.75)
 		(end 176.79 107.75)
@@
 	)
 	(segment
+		(start 121 86.5)
+		(end 117.42 90.08)
+		(width 1.5)
+		(layer "F.Cu")
+		(net "+12V")
+	)
+	(segment
 		(start 136.95 96.65)
 		(end 135.997208 97.602792)
@@
 	)
 	(segment
+		(start 117.5 100.55)
+		(end 123.2 106.25)
+		(width 1.5)
+		(layer "F.Cu")
+		(net "+12V")
+	)
+	(segment
 		(start 176.79 107.75)
 		(end 183.5825 114.5425)
@@
 	)
 	(segment
+		(start 137.12 77.995)
+		(end 137.125 78)
+		(width 1.5)
+		(layer "F.Cu")
+		(net "+12V")
+	)
+	(segment
+		(start 137.12 74.99)
+		(end 137.12 77.995)
+		(width 1.5)
+		(layer "F.Cu")
+		(net "+12V")
+	)
+	(segment
 		(start 142.54 98.25)
 		(end 152.04 107.75)
@@
 	)
 	(segment
+		(start 176.095 115.42)
+		(end 176.29 115.225)
+		(width 1.5)
+		(layer "F.Cu")
+		(net "+5V")
+	)
+	(segment
+		(start 172.79 115.42)
+		(end 176.095 115.42)
+		(width 1.5)
+		(layer "F.Cu")
+		(net "+5V")
+	)
+	(segment
